Commit message: added models

File: PyBullet/models/urdf/blue_book.urdf (robot description, URDF)
Before this commit: robot myfirst, 1 links, 0 joints
Links:
- removed link base_link
- added link tray.SLDPRT, mass 10.8496; collision mesh filename=models/meshes/book/book.STL scale=0.004 0.004 0.004; visual mesh filename=models/meshes/book/book.STL scale=0.004 0.004 0.004

File: PyBullet/models/urdf/box.urdf (robot description, URDF)
Before this commit: robot box, 1 links, 0 joints
Links:
- removed link base_link
- added link box.SLDPRT, mass 13.99; collision mesh filename=models/meshes/box/box.SLDPRT.STL; visual mesh filename=models/meshes/box/box.SLDPRT.STL

File: PyBullet/models/urdf/gray_cube.urdf (robot description, URDF)
Before this commit: robot cube, 1 links, 0 joints
Links:
- link cube-base: mass None -> 2.0

File: PyBullet/models/urdf/sisbot.urdf (robot description, URDF)
Before this commit: robot sisbot, 19 links, 18 joints
Joints:
- joint elbow_joint: limit lower=-3.14159265359 upper=3.14159265359 effort=150.0 velocity=3.15 -> lower=-3.14159265359 upper=3.14159265359 effort=1550.0 velocity=3.15
- joint shoulder_lift_joint: limit lower=-3.14159265359 upper=3.14159265359 effort=150.0 velocity=3.15 -> lower=-3.14159265359 upper=3.14159265359 effort=1550.0 velocity=3.15
- joint wrist_1_joint: limit lower=-3.14159265359 upper=3.14159265359 effort=28.0 velocity=3.2 -> lower=-3.14159265359 upper=3.14159265359 effort=1558.0 velocity=3.2
- joint wrist_2_joint: limit lower=-3.14159265359 upper=3.14159265359 effort=28.0 velocity=3.2 -> lower=-3.14159265359 upper=3.14159265359 effort=1558.0 velocity=3.2
- joint wrist_3_joint: limit lower=-3.14159265359 upper=3.14159265359 effort=28.0 velocity=3.2 -> lower=-3.14159265359 upper=3.14159265359 effort=10055.0 velocity=3.2

File: PyBullet/models/urdf/tray.urdf (robot description, URDF)
Before this commit: robot tray, 1 links, 0 joints
Links:
- removed link tray-base
- added link tray.SLDPRT, mass 0.18496; collision mesh filename=models/meshes/tray/tray.SLDPRT.STL scale=2 2 2; visual mesh filename=models/meshes/tray/tray.SLDPRT.STL scale=2 2 2
