Commit message: added more objects

File: PyBullet/models/urdf/apple.urdf (robot description, URDF)
Before this commit: robot apple, 1 links, 0 joints
Links:
- link base_link: mass 0 -> 5; geometry collision mesh filename=models/meshes/apple/10162_Apple_v01_l3.obj scale=0.0006 0.0007 0.0007; visual mesh filename=models/meshes/apple/10162_Apple_v01_l3.obj scale=0.0007 0.0007 0.0007

File: PyBullet/models/urdf/bottle.urdf (robot description, URDF)
Before this commit: robot Part3.SLDPRT, 1 links, 0 joints
Links:
- link Part3.SLDPRT: mass 0.026721 -> 15.026721; geometry collision mesh filename=models/meshes/bottle/Part3.SLDPRT.STL scale=2 2 2; visual mesh filename=models/meshes/bottle/Part3.SLDPRT.STL scale=2 2 2
