Commit message: added constraints for pick/place/drop

File: PyBullet/models/urdf/box.urdf (robot description, URDF)
Before this commit: robot box.SLDPRT, 1 links, 0 joints
Links:
- link box.SLDPRT: mass 13.99 -> 1.99

Commit message: Added push and a cleaning input example

File: PyBullet/models/urdf/box.urdf (robot description, URDF)
Before this commit: robot box.SLDPRT, 1 links, 0 joints
Links:
- link box.SLDPRT: mass 1.99 -> 15.99

File: PyBullet/models/urdf/sisbot.urdf (robot description, URDF)
Before this commit: robot sisbot, 19 links, 18 joints
Joints:
- joint shoulder_pan_joint: limit lower=-3.14159265359 upper=3.14159265359 effort=150.0 velocity=3.15 -> lower=-3.14159265359 upper=3.14159265359 effort=1550.0 velocity=3.15
