Commit message: updated models

File: PyBullet/models/urdf/book.urdf (robot description, URDF)
Before this commit: robot ball, 1 links, 0 joints
Links:
- link base_link: mass 5 -> 2

File: PyBullet/models/urdf/box.urdf (robot description, URDF)
Before this commit: robot box.SLDPRT, 1 links, 0 joints
Links:
- link box.SLDPRT: mass 15.99 -> 1.99

File: PyBullet/models/urdf/dumpster.urdf (robot description, URDF)
Before this commit: robot ball, 1 links, 0 joints
Links:
- link base_link: mass 5 -> 0
