Commit message: Added stool and related actions of climbing up or down

File: PyBullet/models/urdf/sisbot.urdf (robot description, URDF)
Before this commit: robot sisbot, 19 links, 18 joints
Joints:
- joint shoulder_pan_joint: limit lower=-3.14159265359 upper=3.14159265359 effort=1550.0 velocity=3.15 -> lower=-3.14159265359 upper=3.14159265359 effort=12550.0 velocity=3.15
