Commit message: Made semantic corrections

File: PyBullet/models/urdf/bottle_blue.urdf (robot description, URDF)
Before this commit: robot Part3.SLDPRT, 1 links, 0 joints
Links:
- link Part3.SLDPRT: mass 15.026721 -> 1.026721

File: PyBullet/models/urdf/bottle_gray.urdf (robot description, URDF)
Before this commit: robot Part3.SLDPRT, 1 links, 0 joints
Links:
- link Part3.SLDPRT: mass 15.026721 -> 1.026721

File: PyBullet/models/urdf/bottle_red.urdf (robot description, URDF)
Before this commit: robot Part3.SLDPRT, 1 links, 0 joints
Links:
- link Part3.SLDPRT: mass 15.026721 -> 1.026721
