Commit message: Bug fixes in stick paper goal

File: PyBullet/models/urdf/paper.urdf (robot description, URDF)
Before this commit: robot milk, 1 links, 0 joints
Links:
- link base_link: mass 0.2 -> 0.1

Commit message: Added paper stick data (partial)

File: PyBullet/models/urdf/paper.urdf (robot description, URDF)
Before this commit: robot milk, 1 links, 0 joints
Links:
- link base_link: mass 0.1 -> 0.7
