Commit message: Updated factory objects

File: PyBullet/models/urdf/ramp_tape.urdf (robot description, URDF)
Before this commit: robot banana, 1 links, 0 joints
Links:
- link base_link: geometry visual mesh filename=models/meshes/ramp_tape/ramp_tape.STL scale=10 10 10

File: PyBullet/models/urdf/worktable.urdf (robot description, URDF)
Before this commit: robot worktable.urdf, 1 links, 0 joints
Links:
- link baseLink: mass .6 -> 0
