Commit message: Added fuel action

File: PyBullet/models/urdf/coal.urdf (robot description, URDF)
Before this commit: robot ball, 1 links, 0 joints
Links:
- link base_link: geometry collision mesh filename=models/meshes/coal/Rock1.obj scale=0.012 0.012 0.012; visual mesh filename=models/meshes/coal/Rock1.obj scale=0.012 0.012 0.012
