Commit message: Completed assembly goals
TODO: update datapoint class, update previous datapoints, update graph embedding function, collect data

File: PyBullet/models/urdf/drill.urdf (robot description, URDF)
Before this commit: robot apple, 1 links, 0 joints
Links:
- link base_link: mass .1 -> .5
