Commit message: Climb up on ladder working

File: PyBullet/models/urdf/ladder.urdf (robot description, URDF)
Before this commit: robot apple, 1 links, 0 joints
Links:
- link base_link: mass .1 -> 2; geometry collision mesh filename=models/meshes/stool/stool.obj scale=2 2 1; visual mesh filename=models/meshes/ladder/ladder.stl scale=2 2 2
