Commit message: Added sample datapoints

File: PyBullet/models/urdf/3d_printer.urdf (robot description, URDF)
Before this commit: robot apple, 1 links, 0 joints
Links:
- link base_link: geometry collision mesh filename=models/meshes/3d_printer/3d_printer.obj scale=0.001 0.001 0.001; visual mesh filename=models/meshes/3d_printer/3d_printer.obj scale=0.005 0.005 0.005

File: PyBullet/models/urdf/ladder.urdf (robot description, URDF)
Before this commit: robot apple, 1 links, 0 joints
Links:
- link base_link: geometry collision mesh filename=models/meshes/stool/stool.obj scale=1 1 1; visual mesh filename=models/meshes/ladder/ladder.stl scale=2 2 2

File: PyBullet/models/urdf/worktable.urdf (robot description, URDF)
Before this commit: robot worktable.urdf, 1 links, 0 joints
Links:
- link baseLink: geometry collision mesh filename=models/meshes/worktable/table.obj scale=1.5 0.5 0.6; visual mesh filename=models/meshes/worktable/table.obj scale=0.1 0.1 0.58
