Commit message: Added dataset for goal 1

File: PyBullet/models/urdf/fridge/fridge_back.urdf (robot description, URDF)
Before this commit: robot walls, 1 links, 0 joints
Links:
- link base_link: geometry collision mesh filename=models/meshes/fridge/fridge_back.obj scale=9 9 9; visual mesh filename=models/meshes/fridge/fridge_back.obj scale=10 10 10
