Commit message: Implemented heavy stack checking + added child position to all constraints

File: PyBullet/models/urdf/lift/lift.urdf (robot description, URDF)
Before this commit: robot walls, 1 links, 0 joints
Links:
- link base_link: geometry collision mesh filename=models/meshes/fridge/fridge.obj scale=10 25 10; visual mesh filename=models/meshes/lift/lift.obj scale=10 25 10

File: PyBullet/models/urdf/lift/lift_base.urdf (robot description, URDF)
Before this commit: robot walls, 1 links, 0 joints
Links:
- link base_link: geometry visual mesh filename=models/meshes/lift/lift_base.obj scale=10 10 10

Commit message: Added sample datapoints for factory

File: PyBullet/models/urdf/lift/lift.urdf (robot description, URDF)
Before this commit: robot walls, 1 links, 0 joints
Links:
- link base_link: geometry collision mesh filename=models/meshes/fridge/fridge.obj scale=10 10 10; visual mesh filename=models/meshes/lift/lift.obj scale=10 10 10
